Commit message: g

File: simulation/map20_1/urdf/map20.urdf (robot description, URDF)
Before this commit: robot map25, 1 links, 0 joints
Links:
- removed link map25
- added link map20, mass 19.377943730784; collision mesh filename=package://map20/meshes/map20.STL; visual mesh filename=package://map20/meshes/map20.STL
